Commit message: Added the inertial model of the robot chassis

File: urdf/dd_robot.urdf (robot description, URDF)
Before this commit: robot dd_robot, 3 links, 2 joints
Links:
- link base_link: mass None -> 5

Commit message: Fixed the duplicated name of the construction cones

File: urdf/dd_robot.urdf (robot description, URDF)
Before this commit: robot dd_robot, 3 links, 2 joints
Links:
- link left_wheel: mass None -> 0.5
- link right_wheel: mass None -> 0.5
