Commit message: Added the laser scanner plugin from gazebo (yet to fix the read. ang

File: urdf/gazebo.xacro (robot description, xacro)
@@ -1,4 +1,14 @@
 <?xml version="1.0"?>
 <robot>
+  <gazebo reference="base_link">
+	<material>Gazebo/Blue</material>
+	<pose>0 0 0.3 0 0 0</pose>
+  </gazebo>
+  <gazebo reference="left_wheel">
+	<material>Gazebo/Black</material>
+  </gazebo>
+  <gazebo reference="right_wheel">
+	<material>Gazebo/Black</material>
+  </gazebo>
   <gazebo>
 	<plugin filename="libgazebo_ros_diff_drive.so" name="differential_drive_controller">
@@ -17,13 +27,39 @@
 	</plugin>
   </gazebo>
-  <gazebo reference="base_link">
-	<material>Gazebo/Blue</material>
-	<pose>0 0 0.3 0 0 0</pose>
-  </gazebo>
-  <gazebo reference="left_wheel">
-	<material>Gazebo/Black</material>
-  </gazebo>
-  <gazebo reference="right_wheel">
-	<material>Gazebo/Black</material>
+  <!-- hokuyo -->
+  <gazebo reference="laser_scanner">
+    <sensor type="gpu_ray" name="head_hokuyo_sensor">
+      <pose>0 0 0 0 0 0</pose>
+      <visualize>false</visualize>
+      <update_rate>20</update_rate>
+      <ray>
+        <scan>
+          <horizontal>
+            <samples>720</samples>
+            <resolution>1</resolution>
+            <min_angle>-1.570796</min_angle>
+            <max_angle>1.570796</max_angle>
+          </horizontal>
+        </scan>
+        <range>
+          <min>0.10</min>
+          <max>10.0</max>
+          <resolution>0.01</resolution>
+        </range>
+        <noise>
+          <type>gaussian</type>
+          <!-- Noise parameters based on published spec for Hokuyo laser
+               achieving "+-30mm" accuracy at range < 10m.  A mean of 0.0m and
+               stddev of 0.01m will put 99.7% of samples within 0.03m of the true
+               reading. -->
+          <mean>0.0</mean>
+          <stddev>0.01</stddev>
+        </noise>
+      </ray>
+      <plugin name="gazebo_ros_head_hokuyo_controller" filename="libgazebo_ros_gpu_laser.so">
+        <topicName>/ros_robotics/laser/scan</topicName>
+        <frameName>laser_scanner</frameName>
+      </plugin>
+    </sensor>
   </gazebo>
 </robot>

Commit message: Fixed the wheel's moment of inertia

File: urdf/gazebo.xacro (robot description, xacro)
@@ -18,6 +18,6 @@
 	  <leftJoint>left_joint_wheel</leftJoint>
 	  <rightJoint>right_joint_wheel</rightJoint>
-	  <wheelSeparation>0.2</wheelSeparation>
-	  <wheelDiameter>0.2</wheelDiameter>
+	  <wheelSeparation>0.6</wheelSeparation>
+	  <wheelDiameter>0.3</wheelDiameter>
 	  <torque>0.1</torque>
 	  <commandTopic>cmd_vel</commandTopic>

File: urdf/macros.xacro (robot description, xacro)
@@ -23,6 +23,6 @@
 	  <inertial>
 		<mass value="0.5"/>
-		<inertia ixx="0.01" ixy="0.0" ixz="0.0"
-				 iyy="0.005" iyz="0.0" izz="0.005"/>
+		<inertia ixx="0.003" ixy="0.0" ixz="0.0"
+				 iyy="0.0056" iyz="0.0" izz="0.003"/>
 	  </inertial>
 	</link>
