Commit message: Added xacro files to better manage the robot description

File: urdf/dd_robot.xacro (robot description, xacro)
@@ -1,13 +1,22 @@
 <?xml version = "1.0"?>
-<robot name = "dd_robot">
-  <material name="blue">
-	<color rgba="0.0 0.5 1.0 1.0"/>
-  </material>
-  <material name="white">
-	<color rgba="1.0 1.0 1.0 1.0"/>
-  </material>
-  <material name="black">
-	<color rgba="0.05 0.05 0.05 1.0"/>
-  </material>
+<!-- the xmlns:xacro part is required for the xacro to run properly -->
+<robot name = "dd_robot" xmlns:xacro="http://www.ros.org/wiki/xacro">
+  <xacro:include filename="$(find ros_robotics)/urdf/materials.xacro" />
+  <gazebo>
+	<plugin filename="libgazebo_ros_diff_drive.so" name="differential_drive_controller">
+	  <legacyMode>false</legacyMode>
+	  <alwaysOn>true</alwaysOn>
+	  <updateRate>20</updateRate>
+	  <leftJoint>joint_left_wheel</leftJoint>
+	  <rightJoint>joint_right_wheel</rightJoint>
+	  <wheelSeparation>0.2</wheelSeparation>
+	  <wheelDiameter>0.2</wheelDiameter>
+	  <torque>0.1</torque>
+	  <commandTopic>cmd_vel</commandTopic>
+	  <odometryTopic>odom</odometryTopic>
+	  <odometryFrame>odom</odometryFrame>
+	  <robotBaseFrame>base_link</robotBaseFrame>
+	</plugin>
+  </gazebo>
   <!-- Base link description -->
   <!-- Differently from the sdf standard, the arguments are usually quoted -->
@@ -120,3 +129,13 @@
 	<axis xyz="0 1 0"/>
   </joint>
+  <gazebo reference="base_link">
+	<material>Gazebo/Blue</material>
+	<pose>0 0 0.3 0 0 0</pose>
+  </gazebo>
+  <gazebo reference="left_wheel">
+	<material>Gazebo/Black</material>
+  </gazebo>
+  <gazebo reference="right_wheel">
+	<material>Gazebo/Black</material>
+  </gazebo>
 </robot>

Commit message: Added a macros file for the xacro description

File: urdf/dd_robot.xacro (robot description, xacro)
@@ -3,20 +3,5 @@
 <robot name = "dd_robot" xmlns:xacro="http://www.ros.org/wiki/xacro">
   <xacro:include filename="$(find ros_robotics)/urdf/materials.xacro" />
-  <gazebo>
-	<plugin filename="libgazebo_ros_diff_drive.so" name="differential_drive_controller">
-	  <legacyMode>false</legacyMode>
-	  <alwaysOn>true</alwaysOn>
-	  <updateRate>20</updateRate>
-	  <leftJoint>joint_left_wheel</leftJoint>
-	  <rightJoint>joint_right_wheel</rightJoint>
-	  <wheelSeparation>0.2</wheelSeparation>
-	  <wheelDiameter>0.2</wheelDiameter>
-	  <torque>0.1</torque>
-	  <commandTopic>cmd_vel</commandTopic>
-	  <odometryTopic>odom</odometryTopic>
-	  <odometryFrame>odom</odometryFrame>
-	  <robotBaseFrame>base_link</robotBaseFrame>
-	</plugin>
-  </gazebo>
+  <xacro:include filename="$(find ros_robotics)/urdf/gazebo.xacro" />
   <!-- Base link description -->
   <!-- Differently from the sdf standard, the arguments are usually quoted -->
@@ -129,13 +114,3 @@
 	<axis xyz="0 1 0"/>
   </joint>
-  <gazebo reference="base_link">
-	<material>Gazebo/Blue</material>
-	<pose>0 0 0.3 0 0 0</pose>
-  </gazebo>
-  <gazebo reference="left_wheel">
-	<material>Gazebo/Black</material>
-  </gazebo>
-  <gazebo reference="right_wheel">
-	<material>Gazebo/Black</material>
-  </gazebo>
 </robot>

Commit message: Fixed the xacro errors by using the xacro prefix and + http

File: urdf/dd_robot.xacro (robot description, xacro)
@@ -4,4 +4,5 @@
   <xacro:include filename="$(find ros_robotics)/urdf/materials.xacro" />
   <xacro:include filename="$(find ros_robotics)/urdf/gazebo.xacro" />
+  <xacro:include filename="$(find ros_robotics)/urdf/macros.xacro" />
   <!-- Base link description -->
   <!-- Differently from the sdf standard, the arguments are usually quoted -->
@@ -51,26 +52,5 @@
   </link>
   <!-- Right wheel -->
-  <link name="right_wheel">
-	<visual>
-	  <origin xyz="0 0 0" rpy="1.570795 0 0" />
-	  <geometry>
-		<cylinder length="0.1" radius="0.2" />
-	  </geometry>
-	  <material name="black"/>
-	</visual>
-	<!-- Right wheel collision -->
-	<collision>
-	  <origin xyz="0 0 0" rpy="1.570795 0 0"/>
-	  <geometry>
-		<cylinder length="0.1" radius="0.2"/>
-	  </geometry>
-	</collision>
-	<!-- Right wheel inertial model -->
-	<inertial>
-	  <mass value="0.5"/>
-	  <inertia ixx="0.01" ixy="0.0" ixz="0.0"
-			   iyy="0.005" iyz="0.0" izz="0.005"/>
-	</inertial>
-  </link>
+  <xacro:link_wheel name="right_wheel"/>
   <!-- The joint origin is defined in regards to the base_link reference (in this case, "0 0 0");
 		hence, the origin of the wheel attached to it indicates, from the origin of the join, where
@@ -83,29 +63,9 @@
 	<axis xyz="0 1 0"/>
   </joint>
+  <!-- Left wheel -->
+  <xacro:link_wheel name="left_wheel"/>
   <!-- left wheel -->
   <!-- The origin of the wheel needs to be the same as the one for the base link
 		for easier desiging of the robot -->
-  <link name="left_wheel">
-	<visual>
-	  <origin xyz="0 0 0" rpy="1.570795 0 0" />
-	  <geometry>
-		<cylinder length="0.1" radius="0.2" />
-	  </geometry>
-	  <material name="black"/>
-	</visual>
-	<!-- Left wheel collision -->
-	<collision>
-	  <origin xyz="0 0 0" rpy="1.570795 0 0"/>
-	  <geometry>
-		<cylinder length="0.1" radius="0.2"/>
-	  </geometry>
-	</collision>
-	<!-- Left wheel inertial model -->
-	<inertial>
-	  <mass value="0.5"/>
-	  <inertia ixx="0.01" ixy="0.0" ixz="0.0"
-			   iyy="0.005" iyz="0.0" izz="0.005"/>
-	</inertial>
-  </link>
   <joint name="joint_left_wheel" type="continuous">
 	<parent link="base_link"/>

File: urdf/macros.xacro (robot description, xacro)
@@ -1,28 +1,28 @@
 <?xml version="1.0"?>
-<robot>
-  <macro name="link_wheel" params="name">
-  <!-- Generic wheel -->
-  <link name="${name}">
-	<visual>
-	  <origin xyz="0 0 0" rpy="1.570795 0 0" />
-	  <geometry>
-		<cylinder length="0.1" radius="0.2" />
-	  </geometry>
-	  <material name="black"/>
-	</visual>
-	<!-- Generic wheel collision -->
-	<collision>
-	  <origin xyz="0 0 0" rpy="1.570795 0 0"/>
-	  <geometry>
-		<cylinder length="0.1" radius="0.2"/>
-	  </geometry>
-	</collision>
-	<!-- Generic wheel inertial model -->
-	<inertial>
-	  <mass value="0.5"/>
-	  <inertia ixx="0.01" ixy="0.0" ixz="0.0"
-			   iyy="0.005" iyz="0.0" izz="0.005"/>
-	</inertial>
-  </link>
-  </macro>
+<robot xmlns:xacro="http://www.ros.org/wiki/xacro">
+  <xacro:macro name="link_wheel" params="name">
+	<!-- Generic wheel -->
+	<link name="${name}">
+	  <visual>
+		<origin xyz="0 0 0" rpy="1.570795 0 0" />
+		<geometry>
+		  <cylinder length="0.1" radius="0.2" />
+		</geometry>
+		<material name="black"/>
+	  </visual>
+	  <!-- Generic wheel collision -->
+	  <collision>
+		<origin xyz="0 0 0" rpy="1.570795 0 0"/>
+		<geometry>
+		  <cylinder length="0.1" radius="0.2"/>
+		</geometry>
+	  </collision>
+	  <!-- Generic wheel inertial model -->
+	  <inertial>
+		<mass value="0.5"/>
+		<inertia ixx="0.01" ixy="0.0" ixz="0.0"
+				 iyy="0.005" iyz="0.0" izz="0.005"/>
+	  </inertial>
+	</link>
+  </xacro:macro>
 </robot>

Commit message: "macrorized" the wheel and the joints, but teleop_twist isn't working

File: urdf/dd_robot.xacro (robot description, xacro)
@@ -53,24 +53,13 @@
   <!-- Right wheel -->
   <xacro:link_wheel name="right_wheel"/>
-  <!-- The joint origin is defined in regards to the base_link reference (in this case, "0 0 0");
-		hence, the origin of the wheel attached to it indicates, from the origin of the join, where
-		the wheel will be drawn. To check this out, change the wheel's origin to 0.3 and leave the
-		joint origin as is.-->
-  <joint name="joint_right_wheel" type="continuous">
-	<parent link="base_link"/>
-	<child link="right_wheel"/>
-	<origin xyz="0 -0.30 0.025" rpy="0 0 0" />
-	<axis xyz="0 1 0"/>
-  </joint>
+  <xacro:joint_wheel name="right" child="right_wheel" x="0" y="-0.30" z="0.025"/>
   <!-- Left wheel -->
   <xacro:link_wheel name="left_wheel"/>
-  <!-- left wheel -->
-  <!-- The origin of the wheel needs to be the same as the one for the base link
-		for easier desiging of the robot -->
-  <joint name="joint_left_wheel" type="continuous">
-	<parent link="base_link"/>
-	<child link="left_wheel"/>
-	<origin xyz="0 0.30 0.025" rpy="0 0 0" />
-	<axis xyz="0 1 0"/>
-  </joint>
+  <xacro:joint_wheel name="left" child="left_wheel" x="0" y="0.30" z="0.025"/>
+  <!-- <joint name="joint_left_wheel" type="continuous"> -->
+  <!-- 	<parent link="base_link"/> -->
+  <!-- 	<child link="left_wheel"/> -->
+  <!-- 	<origin xyz="0 0.30 0.025" rpy="0 0 0" /> -->
+  <!-- 	<axis xyz="0 1 0"/> -->
+  <!-- </joint> -->
 </robot>

File: urdf/macros.xacro (robot description, xacro)
@@ -1,4 +1,6 @@
 <?xml version="1.0"?>
 <robot xmlns:xacro="http://www.ros.org/wiki/xacro">
+  <!-- The origin of the wheel needs to be the same as the one for the base link
+		for easier desiging of the robot -->
   <xacro:macro name="link_wheel" params="name">
 	<!-- Generic wheel -->
@@ -26,3 +28,15 @@
 	</link>
   </xacro:macro>
+  <!-- The joint origin is defined in regards to the base_link reference (in this case, "0 0 0");
+		hence, the origin of the wheel attached to it indicates, from the origin of the join, where
+		the wheel will be drawn. To check this out, change the wheel's origin to 0.3 and leave the
+		joint origin as is.-->
+  <xacro:macro name="joint_wheel" params="name child x y z">
+	<joint name="${name}_joint_wheel" type="continuous">
+	  <parent link="base_link"/>
+	  <child link="${child}"/>
+	  <origin xyz="${x} ${y} ${z}" rpy="0 0 0" />
+	  <axis xyz="0 1 0"/>
+	</joint>
+  </xacro:macro>
 </robot>

Commit message: Updated the rviz launch file to allow the usage of xacros

File: urdf/dd_robot.xacro (robot description, xacro)
@@ -57,9 +57,3 @@
   <xacro:link_wheel name="left_wheel"/>
   <xacro:joint_wheel name="left" child="left_wheel" x="0" y="0.30" z="0.025"/>
-  <!-- <joint name="joint_left_wheel" type="continuous"> -->
-  <!-- 	<parent link="base_link"/> -->
-  <!-- 	<child link="left_wheel"/> -->
-  <!-- 	<origin xyz="0 0.30 0.025" rpy="0 0 0" /> -->
-  <!-- 	<axis xyz="0 1 0"/> -->
-  <!-- </joint> -->
 </robot>

Commit message: Added a laser scanner link to the urdf model of the robot I should, maybe, reduce the wheels size

File: urdf/dd_robot.xacro (robot description, xacro)
@@ -51,4 +51,30 @@
 	</inertial>
   </link>
+  <link name="laser_scanner">
+	<visual>
+	  <origin xyz="0 0 0" rpy="0 0 0"/>
+	  <geometry>
+		<cylinder length="0.1" radius="0.1"/>
+	  </geometry>
+	  <material name="white"/>
+	</visual>
+	<inertial>
+	  <origin xyz="0 0 0" rpy="0 0 0"/>
+	  <mass value="0.5"/>
+	  <xacro:cylinder_inertia mass="0.5" r="0.1" l="0.2"/>
+	</inertial>
+	<collision>
+	  <origin xyz="0 0 0" rpy="0 0 0"/>
+	  <geometry>
+		<cylinder length="0.1" radius="0.1"/>
+	  </geometry>
+	</collision>
+  </link>
+  <joint name="laser_scanner_joint" type="continuous">
+	<parent link="base_link"/>
+	<child link="laser_scanner"/>
+	<origin xyz="0.1 0 0.175" rpy="0 0 0"/>
+	<axis xyz="0 0 1"/>
+  </joint>
   <!-- Right wheel -->
   <xacro:link_wheel name="right_wheel"/>

File: urdf/macros.xacro (robot description, xacro)
@@ -40,3 +40,9 @@
 	</joint>
   </xacro:macro>
+  <!-- https://en.wikipedia.org/wiki/List_of_moments_of_inertia#List_of_3D_inertia_tensors -->
+  <xacro:macro name="cylinder_inertia" params="mass r l">
+	<inertia ixx="${mass * (3 * r * r + l * l) / 12}" ixy="0.0" ixz="0.0"
+			 iyy="${mass * (3 * r * r + l * l) / 12}" iyz="0.0"
+			 izz="${mass *  (r * r) / 2}"/>
+  </xacro:macro>
 </robot>

Commit message: Modified the wheel's position and their size

File: urdf/dd_robot.xacro (robot description, xacro)
@@ -79,7 +79,7 @@
   <!-- Right wheel -->
   <xacro:link_wheel name="right_wheel"/>
-  <xacro:joint_wheel name="right" child="right_wheel" x="0" y="-0.30" z="0.025"/>
+  <xacro:joint_wheel name="right" child="right_wheel" x="0" y="-0.30" z="-0.025"/>
   <!-- Left wheel -->
   <xacro:link_wheel name="left_wheel"/>
-  <xacro:joint_wheel name="left" child="left_wheel" x="0" y="0.30" z="0.025"/>
+  <xacro:joint_wheel name="left" child="left_wheel" x="0" y="0.30" z="-0.025"/>
 </robot>

File: urdf/gazebo.xacro (robot description, xacro)
@@ -38,6 +38,6 @@
             <samples>720</samples>
             <resolution>1</resolution>
-            <min_angle>-1.570796</min_angle>
-            <max_angle>1.570796</max_angle>
+            <min_angle>-3.14159</min_angle>
+            <max_angle>3.14159</max_angle>
           </horizontal>
         </scan>

File: urdf/macros.xacro (robot description, xacro)
@@ -9,5 +9,5 @@
 		<origin xyz="0 0 0" rpy="1.570795 0 0" />
 		<geometry>
-		  <cylinder length="0.1" radius="0.2" />
+		  <cylinder length="0.1" radius="0.15" />
 		</geometry>
 		<material name="black"/>
@@ -17,5 +17,5 @@
 		<origin xyz="0 0 0" rpy="1.570795 0 0"/>
 		<geometry>
-		  <cylinder length="0.1" radius="0.2"/>
+		  <cylinder length="0.1" radius="0.15"/>
 		</geometry>
 	  </collision>

Commit message: Changed the chassis size and the mmts of inertia

File: urdf/dd_robot.xacro (robot description, xacro)
@@ -11,5 +11,5 @@
 	  <origin xyz = "0 0 0" rpy = "0 0 0 " />
 	  <geometry>
-		<box size = "0.5 0.5 0.25" />
+		<box size = "0.8 0.5 0.25" />
 	  </geometry>
 	  <material name="blue"/>
@@ -19,5 +19,5 @@
 	  <origin xyz="0 0 0" rpy="0 0 0"/>
 	  <geometry>
-		<box size="0.5 0.5 0.25"/>
+		<box size="0.8 0.5 0.25"/>
 	  </geometry>
 	</collision>
@@ -25,6 +25,8 @@
 	<inertial>
 	  <mass value="5"/>
-	  <inertia ixx="0.13" ixy="0.0" ixz="0.0"
-			   iyy="0.21" iyz="0.0" izz="0.13"/>
+	  <inertia ixx="0.29" ixy="0.0" ixz="0.0"
+	  		   iyy="0.37" iyz="0.0" izz="0.13"/>
+	  <!-- <inertia ixx="0.13" ixy="0.0" ixz="0.0" -->
+	  <!-- 		   iyy="0.21" iyz="0.0" izz="0.13"/> -->
 	</inertial>
 	<!-- Caster -->
@@ -32,5 +34,5 @@
 		 it would need a joint to attach it to the base link -->
 	<visual name="caster">
-	  <origin xyz="0.2 0 -0.125" rpy="0 0 0"/>
+	  <origin xyz="0.35 0 -0.125" rpy="0 0 0"/>
 	  <geometry>
 		<sphere radius="0.05"/>
@@ -40,5 +42,5 @@
 	<!-- Caster collision -->
 	<collision>
-	  <origin xyz="0.2 0 -0.125" rpy="0 0 0"/>
+	  <origin xyz="0.35 0 -0.125" rpy="0 0 0"/>
 	  <geometry>
 		<sphere radius="0.05"/>
@@ -79,7 +81,7 @@
   <!-- Right wheel -->
   <xacro:link_wheel name="right_wheel"/>
-  <xacro:joint_wheel name="right" child="right_wheel" x="0" y="-0.30" z="-0.025"/>
+  <xacro:joint_wheel name="right" child="right_wheel" x="-0.25" y="-0.30" z="-0.025"/>
   <!-- Left wheel -->
   <xacro:link_wheel name="left_wheel"/>
-  <xacro:joint_wheel name="left" child="left_wheel" x="0" y="0.30" z="-0.025"/>
+  <xacro:joint_wheel name="left" child="left_wheel" x="-0.25" y="0.30" z="-0.025"/>
 </robot>

File: urdf/gazebo.xacro (robot description, xacro)
@@ -31,4 +31,5 @@
     <sensor type="gpu_ray" name="head_hokuyo_sensor">
       <pose>0 0 0 0 0 0</pose>
+	  <!-- This parameter controls wether we can see the laser or not -->
       <visualize>false</visualize>
       <update_rate>20</update_rate>

Commit message: Fixed the CMakeLists file and added TF broad/list topics

File: urdf/dd_robot.xacro (robot description, xacro)
@@ -11,5 +11,5 @@
 	  <origin xyz = "0 0 0" rpy = "0 0 0 " />
 	  <geometry>
-		<box size = "0.8 0.5 0.25" />
+		<box size = "0.5 0.5 0.25" />
 	  </geometry>
 	  <material name="blue"/>
@@ -19,5 +19,5 @@
 	  <origin xyz="0 0 0" rpy="0 0 0"/>
 	  <geometry>
-		<box size="0.8 0.5 0.25"/>
+		<box size="0.5 0.5 0.25"/>
 	  </geometry>
 	</collision>
@@ -25,8 +25,8 @@
 	<inertial>
 	  <mass value="5"/>
-	  <inertia ixx="0.29" ixy="0.0" ixz="0.0"
-	  		   iyy="0.37" iyz="0.0" izz="0.13"/>
-	  <!-- <inertia ixx="0.13" ixy="0.0" ixz="0.0" -->
-	  <!-- 		   iyy="0.21" iyz="0.0" izz="0.13"/> -->
+	  <!-- <inertia ixx="0.29" ixy="0.0" ixz="0.0" -->
+	  <!-- 		   iyy="0.37" iyz="0.0" izz="0.13"/> -->
+	  <inertia ixx="0.13" ixy="0.0" ixz="0.0"
+	  		   iyy="0.13" iyz="0.0" izz="0.208"/>
 	</inertial>
 	<!-- Caster -->
@@ -34,5 +34,5 @@
 		 it would need a joint to attach it to the base link -->
 	<visual name="caster">
-	  <origin xyz="0.35 0 -0.125" rpy="0 0 0"/>
+	  <origin xyz="0.2 0 -0.125" rpy="0 0 0"/>
 	  <geometry>
 		<sphere radius="0.05"/>
@@ -42,5 +42,5 @@
 	<!-- Caster collision -->
 	<collision>
-	  <origin xyz="0.35 0 -0.125" rpy="0 0 0"/>
+	  <origin xyz="0.2 0 -0.125" rpy="0 0 0"/>
 	  <geometry>
 		<sphere radius="0.05"/>
@@ -81,7 +81,7 @@
   <!-- Right wheel -->
   <xacro:link_wheel name="right_wheel"/>
-  <xacro:joint_wheel name="right" child="right_wheel" x="-0.25" y="-0.30" z="-0.025"/>
+  <xacro:joint_wheel name="right" child="right_wheel" x="-0.1" y="-0.30" z="-0.025"/>
   <!-- Left wheel -->
   <xacro:link_wheel name="left_wheel"/>
-  <xacro:joint_wheel name="left" child="left_wheel" x="-0.25" y="0.30" z="-0.025"/>
+  <xacro:joint_wheel name="left" child="left_wheel" x="-0.1" y="0.30" z="-0.025"/>
 </robot>

Commit message: Fixed the differential driver parameters

File: urdf/dd_robot.xacro (robot description, xacro)
@@ -11,5 +11,5 @@
 	  <origin xyz = "0 0 0" rpy = "0 0 0 " />
 	  <geometry>
-		<box size = "0.5 0.5 0.25" />
+		<box size = "0.8 0.5 0.25" />
 	  </geometry>
 	  <material name="blue"/>
@@ -19,5 +19,5 @@
 	  <origin xyz="0 0 0" rpy="0 0 0"/>
 	  <geometry>
-		<box size="0.5 0.5 0.25"/>
+		<box size="0.8 0.5 0.25"/>
 	  </geometry>
 	</collision>
@@ -25,14 +25,14 @@
 	<inertial>
 	  <mass value="5"/>
-	  <!-- <inertia ixx="0.29" ixy="0.0" ixz="0.0" -->
-	  <!-- 		   iyy="0.37" iyz="0.0" izz="0.13"/> -->
 	  <inertia ixx="0.13" ixy="0.0" ixz="0.0"
-	  		   iyy="0.13" iyz="0.0" izz="0.208"/>
+	  		   iyy="0.29" iyz="0.0" izz="0.371"/>
+	  <!-- <inertia ixx="0.13" ixy="0.0" ixz="0.0" -->
+	  <!-- 		   iyy="0.13" iyz="0.0" izz="0.208"/> -->
 	</inertial>
-	<!-- Caster -->
+	<!-- Front Caster -->
 	<!-- The caster is inside of the base link. I couldn't create it a link because
 		 it would need a joint to attach it to the base link -->
 	<visual name="caster">
-	  <origin xyz="0.2 0 -0.125" rpy="0 0 0"/>
+	  <origin xyz="0.35 0 -0.125" rpy="0 0 0"/>
 	  <geometry>
 		<sphere radius="0.05"/>
@@ -42,5 +42,5 @@
 	<!-- Caster collision -->
 	<collision>
-	  <origin xyz="0.2 0 -0.125" rpy="0 0 0"/>
+	  <origin xyz="0.35 0 -0.125" rpy="0 0 0"/>
 	  <geometry>
 		<sphere radius="0.05"/>
@@ -81,7 +81,7 @@
   <!-- Right wheel -->
   <xacro:link_wheel name="right_wheel"/>
-  <xacro:joint_wheel name="right" child="right_wheel" x="-0.1" y="-0.30" z="-0.025"/>
+  <xacro:joint_wheel name="right" child="right_wheel" x="-0.35" y="-0.30" z="-0.025"/>
   <!-- Left wheel -->
   <xacro:link_wheel name="left_wheel"/>
-  <xacro:joint_wheel name="left" child="left_wheel" x="-0.1" y="0.30" z="-0.025"/>
+  <xacro:joint_wheel name="left" child="left_wheel" x="-0.35" y="0.30" z="-0.025"/>
 </robot>

Commit message: Modified the chassis shape and the caster's position

File: urdf/dd_robot.xacro (robot description, xacro)
@@ -11,5 +11,5 @@
 	  <origin xyz = "0 0 0" rpy = "0 0 0 " />
 	  <geometry>
-		<box size = "0.8 0.5 0.25" />
+		<box size = ".4 .2 .1" />
 	  </geometry>
 	  <material name="blue"/>
@@ -17,16 +17,17 @@
 	<!-- Chassis collision -->
 	<collision>
-	  <origin xyz="0 0 0" rpy="0 0 0"/>
+	  <!-- <origin xyz="0 0 0" rpy="0 0 0"/> -->
 	  <geometry>
-		<box size="0.8 0.5 0.25"/>
+		<box size=".4 .2 .1"/>
 	  </geometry>
 	</collision>
 	<!-- Inertial properties of the chassis -->
 	<inertial>
-	  <mass value="5"/>
-	  <inertia ixx="0.13" ixy="0.0" ixz="0.0"
-	  		   iyy="0.29" iyz="0.0" izz="0.371"/>
+	  <mass value="10"/>
+	  <origin xyz="0.0 0 0.1" rpy = "0 0 0" />
 	  <!-- <inertia ixx="0.13" ixy="0.0" ixz="0.0" -->
-	  <!-- 		   iyy="0.13" iyz="0.0" izz="0.208"/> -->
+	  <!-- 		   iyy="0.29" iyz="0.0" izz="0.371"/> -->
+	  <inertia ixx = "0.042" ixy = "0.0" ixz = "0.0"
+	  		   iyy = "0.142" iyz = "0.0" izz = "0.167"/>
 	</inertial>
 	<!-- Front Caster -->
@@ -34,5 +35,5 @@
 		 it would need a joint to attach it to the base link -->
 	<visual name="caster">
-	  <origin xyz="0.35 0 -0.125" rpy="0 0 0"/>
+	  <origin xyz=".15 0 -0.05" rpy="0 0 0"/>
 	  <geometry>
 		<sphere radius="0.05"/>
@@ -41,9 +42,19 @@
 	</visual>
 	<!-- Caster collision -->
-	<collision>
-	  <origin xyz="0.35 0 -0.125" rpy="0 0 0"/>
+	<collision name='caster_collision'>
+	  <origin xyz="0.15 0 -0.05" rpy="0 0 0"/>
 	  <geometry>
 		<sphere radius="0.05"/>
 	  </geometry>
+	  <surface>
+		<friction>
+		  <ode>
+			<mu>0</mu>
+			<mu2>0</mu2>
+			<slip1>1.0</slip1>
+			<slip2>1.0</slip2>
+		  </ode>
+		</friction>
+	  </surface>
 	</collision>
 	<inertial>
