Commit message: Fixed the cylinder_inertias: were missing the <inertial> tag

File: urdf/dd_robot.xacro (robot description, xacro)
@@ -75,5 +75,5 @@
 	  <origin xyz="0 0 0" rpy="0 0 0"/>
 	  <mass value="0.5"/>
-	  <xacro:cylinder_inertia mass="0.5" r="0.1" l="0.2"/>
+	  <xacro:cylinder_inertia_z_axis mass="0.5" r="0.1" l="0.1"/>
 	</inertial>
 	<collision>
@@ -87,12 +87,12 @@
 	<parent link="base_link"/>
 	<child link="laser_scanner"/>
-	<origin xyz="0.1 0 0.175" rpy="0 0 0"/>
+	<origin xyz="0.0 0.0 0.175" rpy="0 0 0"/>
 	<axis xyz="0 0 1"/>
   </joint>
   <!-- Right wheel -->
   <xacro:link_wheel name="right_wheel"/>
-  <xacro:joint_wheel name="right" child="right_wheel" x="-0.35" y="-0.30" z="-0.025"/>
+  <xacro:joint_wheel name="right" child="right_wheel" x="-0.1" y="-0.15" z="0.0"/>
   <!-- Left wheel -->
   <xacro:link_wheel name="left_wheel"/>
-  <xacro:joint_wheel name="left" child="left_wheel" x="-0.35" y="0.30" z="-0.025"/>
+  <xacro:joint_wheel name="left" child="left_wheel" x="-0.1" y="0.15" z="0.0"/>
 </robot>

File: urdf/macros.xacro (robot description, xacro)
@@ -1,6 +1,23 @@
 <?xml version="1.0"?>
 <robot xmlns:xacro="http://www.ros.org/wiki/xacro">
+  <!-- https://en.wikipedia.org/wiki/List_of_moments_of_inertia#List_of_3D_inertia_tensors -->
+  <xacro:macro name="cylinder_inertia_z_axis" params="mass r l">
+	<inertial>
+	  <mass value="${mass}"/>
+	  <inertia ixx="${mass * (3 * r * r + l * l) / 12}" ixy="0.0" ixz="0.0"
+			   iyy="${mass * (3 * r * r + l * l) / 12}" iyz="0.0"
+			   izz="${mass *  (r * r) / 2}"/>
+	</inertial>
+  </xacro:macro>
+  <xacro:macro name="cylinder_inertia_y_axis" params="mass r l">
+	<inertial>
+	  <mass value="${mass}"/>
+	  <inertia ixx="${mass * (3 * r * r + l * l) / 12}" ixy="0.0" ixz="0.0"
+			   iyy="${mass *  (r * r) / 2}" iyz="0.0"
+			   izz="${mass * (3 * r * r + l * l) / 12}"/>
+	</inertial>
+  </xacro:macro>
   <!-- The origin of the wheel needs to be the same as the one for the base link
-		for easier desiging of the robot -->
+	   for easier desiging of the robot -->
   <xacro:macro name="link_wheel" params="name">
 	<!-- Generic wheel -->
@@ -9,5 +26,5 @@
 		<origin xyz="0 0 0" rpy="1.570795 0 0" />
 		<geometry>
-		  <cylinder length="0.1" radius="0.15" />
+		  <cylinder length="0.05" radius="0.1" />
 		</geometry>
 		<material name="black"/>
@@ -17,13 +34,16 @@
 		<origin xyz="0 0 0" rpy="1.570795 0 0"/>
 		<geometry>
-		  <cylinder length="0.1" radius="0.15"/>
+		  <cylinder length="0.05" radius="0.1"/>
 		</geometry>
 	  </collision>
+	  <xacro:cylinder_inertia_y_axis mass="5" r="0.1" l="0.05"/>
 	  <!-- Generic wheel inertial model -->
-	  <inertial>
-		<mass value="0.5"/>
-		<inertia ixx="0.003" ixy="0.0" ixz="0.0"
-				 iyy="0.0056" iyz="0.0" izz="0.003"/>
-	  </inertial>
+	  <!-- I've replaced this by a macro of cylinder inertial rotating -->
+	  <!-- on the y axis. -->
+	  <!-- <inertial> -->
+	  <!-- 	<mass value="5"/> -->
+	  <!-- 	<inertia ixx="0.003" ixy="0.0" ixz="0.0" -->
+	  <!-- 			 iyy="0.025" iyz="0.0" izz="0.003"/> -->
+	  <!-- </inertial> -->
 	</link>
   </xacro:macro>
@@ -40,9 +60,3 @@
 	</joint>
   </xacro:macro>
-  <!-- https://en.wikipedia.org/wiki/List_of_moments_of_inertia#List_of_3D_inertia_tensors -->
-  <xacro:macro name="cylinder_inertia" params="mass r l">
-	<inertia ixx="${mass * (3 * r * r + l * l) / 12}" ixy="0.0" ixz="0.0"
-			 iyy="${mass * (3 * r * r + l * l) / 12}" iyz="0.0"
-			 izz="${mass *  (r * r) / 2}"/>
-  </xacro:macro>
 </robot>

Commit message: Chaged the shape of the laser scanner and some colors

File: urdf/dd_robot.xacro (robot description, xacro)
@@ -68,17 +68,13 @@
 	  <origin xyz="0 0 0" rpy="0 0 0"/>
 	  <geometry>
-		<cylinder length="0.1" radius="0.1"/>
+		<cylinder length="0.05" radius="0.05"/>
 	  </geometry>
-	  <material name="white"/>
+	  <material name="black"/>
 	</visual>
-	<inertial>
-	  <origin xyz="0 0 0" rpy="0 0 0"/>
-	  <mass value="0.5"/>
-	  <xacro:cylinder_inertia_z_axis mass="0.5" r="0.1" l="0.1"/>
-	</inertial>
+	<xacro:cylinder_inertia_z_axis mass="0.5" r="0.05" l="0.05"/>
 	<collision>
 	  <origin xyz="0 0 0" rpy="0 0 0"/>
 	  <geometry>
-		<cylinder length="0.1" radius="0.1"/>
+		<cylinder length="0.05" radius="0.05"/>
 	  </geometry>
 	</collision>
@@ -87,5 +83,5 @@
 	<parent link="base_link"/>
 	<child link="laser_scanner"/>
-	<origin xyz="0.0 0.0 0.175" rpy="0 0 0"/>
+	<origin xyz="0.0 0.0 0.05" rpy="0 0 0"/>
 	<axis xyz="0 0 1"/>
   </joint>

File: urdf/macros.xacro (robot description, xacro)
@@ -28,5 +28,5 @@
 		  <cylinder length="0.05" radius="0.1" />
 		</geometry>
-		<material name="black"/>
+		<material name="white"/>
 	  </visual>
 	  <!-- Generic wheel collision -->

Commit message: Minor fixes + move the laser scanner a bit upwards

File: urdf/dd_robot.xacro (robot description, xacro)
@@ -68,13 +68,13 @@
 	  <origin xyz="0 0 0" rpy="0 0 0"/>
 	  <geometry>
-		<cylinder length="0.05" radius="0.05"/>
+		<cylinder length="0.1" radius="0.05"/>
 	  </geometry>
 	  <material name="black"/>
 	</visual>
-	<xacro:cylinder_inertia_z_axis mass="0.5" r="0.05" l="0.05"/>
+	<xacro:cylinder_inertia_z_axis mass="0.5" r="0.05" l="0.1"/>
 	<collision>
 	  <origin xyz="0 0 0" rpy="0 0 0"/>
 	  <geometry>
-		<cylinder length="0.05" radius="0.05"/>
+		<cylinder length="0.1" radius="0.05"/>
 	  </geometry>
 	</collision>
@@ -83,5 +83,5 @@
 	<parent link="base_link"/>
 	<child link="laser_scanner"/>
-	<origin xyz="0.0 0.0 0.05" rpy="0 0 0"/>
+	<origin xyz="0.0 0.0 0.1" rpy="0 0 0"/>
 	<axis xyz="0 0 1"/>
   </joint>

File: urdf/gazebo.xacro (robot description, xacro)
@@ -6,7 +6,10 @@
   </gazebo>
   <gazebo reference="left_wheel">
-	<material>Gazebo/Black</material>
+	<material>Gazebo/White</material>
   </gazebo>
   <gazebo reference="right_wheel">
+	<material>Gazebo/White</material>
+  </gazebo>
+  <gazebo reference="laser_scanner">
 	<material>Gazebo/Black</material>
   </gazebo>

Commit message: Added a green material color and adding a camera link

File: urdf/dd_robot.xacro (robot description, xacro)
@@ -5,4 +5,6 @@
   <xacro:include filename="$(find ros_robotics)/urdf/gazebo.xacro" />
   <xacro:include filename="$(find ros_robotics)/urdf/macros.xacro" />
+  <xacro:property name="cameraSize" value="0.05"/>
+  <xacro:property name="cameraMass" value="0.1"/>
   <!-- Base link description -->
   <!-- Differently from the sdf standard, the arguments are usually quoted -->
@@ -64,4 +66,12 @@
 	</inertial>
   </link>
+  <link name="camera">
+	<visual>
+	  <origin xyz="0 0 0" rpy="0 0 0"/>
+	  <geometry>
+		<box size="${cameraSize} ${cameraSize} ${cameraSize}"/>
+	  </geometry>
+	  <material name="green"/>
+	</visual>
   <link name="laser_scanner">
 	<visual>

File: urdf/materials.xacro (robot description, xacro)
@@ -10,3 +10,6 @@
 	<color rgba="0.05 0.05 0.05 1.0"/>
   </material>
+  <material name="green">
+	<color rgba="0.05 1.0 0.05"/>
+  </material>
 </robot>

Commit message: Added the camera urdf and plugin to the model

File: urdf/dd_robot.xacro (robot description, xacro)
@@ -66,5 +66,5 @@
 	</inertial>
   </link>
-  <link name="camera">
+  <link name="camera_link">
 	<visual>
 	  <origin xyz="0 0 0" rpy="0 0 0"/>
@@ -74,4 +74,21 @@
 	  <material name="green"/>
 	</visual>
+	<collision>
+	  <origin xyz="0 0 0" rpy="0 0 0"/>
+	  <geometry>
+		<box size="${cameraSize} ${cameraSize} ${cameraSize}"/>
+	  </geometry>
+	</collision>
+	<inertial>
+	  <mass value="${cameraMass}"/>
+	  <inertia ixx="1e-6" ixy="0" ixz="0" iyy="1e-6" iyz="0" izz="1e-6"/>
+	</inertial>
+  </link>
+  <joint name="camera_joint" type="fixed">
+	<parent link="base_link"/>
+	<child link="camera_link"/>
+	<origin xyz="0.2 0.0 0.0" rpy="0 0 0"/>
+	<axis xyz="0 1 0"/>
+  </joint>
   <link name="laser_scanner">
 	<visual>

File: urdf/gazebo.xacro (robot description, xacro)
@@ -29,4 +29,44 @@
 	  <robotBaseFrame>base_link</robotBaseFrame>
 	</plugin>
+  </gazebo>
+  <!-- camera -->
+  <gazebo reference="camera_link">
+    <sensor type="camera" name="camera1">
+      <update_rate>30.0</update_rate>
+      <camera name="head">
+        <horizontal_fov>1.3962634</horizontal_fov>
+        <image>
+          <width>800</width>
+          <height>800</height>
+          <format>R8G8B8</format>
+        </image>
+        <clip>
+          <near>0.02</near>
+          <far>300</far>
+        </clip>
+        <noise>
+          <type>gaussian</type>
+          <!-- Noise is sampled independently per pixel on each frame.
+               That pixel's noise value is added to each of its color
+               channels, which at that point lie in the range [0,1]. -->
+          <mean>0.0</mean>
+          <stddev>0.007</stddev>
+        </noise>
+      </camera>
+      <plugin name="camera_controller" filename="libgazebo_ros_camera.so">
+        <alwaysOn>true</alwaysOn>
+        <updateRate>0.0</updateRate>
+        <cameraName>ddrobot/camera1</cameraName>
+        <imageTopicName>image_raw</imageTopicName>
+        <cameraInfoTopicName>camera_info</cameraInfoTopicName>
+        <frameName>camera_link</frameName>
+        <hackBaseline>0.07</hackBaseline>
+        <distortionK1>0.0</distortionK1>
+        <distortionK2>0.0</distortionK2>
+        <distortionK3>0.0</distortionK3>
+        <distortionT1>0.0</distortionT1>
+        <distortionT2>0.0</distortionT2>
+      </plugin>
+    </sensor>
   </gazebo>
   <!-- hokuyo -->

Commit message: Increased the robot's mass from 10 to 15 to prevent wobbling (inertia

File: urdf/dd_robot.xacro (robot description, xacro)
@@ -26,5 +26,5 @@
 	<!-- Inertial properties of the chassis -->
 	<inertial>
-	  <mass value="10"/>
+	  <mass value="15"/>
 	  <origin xyz="0.0 0 0.1" rpy = "0 0 0" />
 	  <!-- <inertia ixx="0.13" ixy="0.0" ixz="0.0" -->

Commit message: Tweaked the inertia to prevent the robot from wobbling

File: urdf/dd_robot.xacro (robot description, xacro)
@@ -28,8 +28,9 @@
 	  <mass value="15"/>
 	  <origin xyz="0.0 0 0.1" rpy = "0 0 0" />
-	  <!-- <inertia ixx="0.13" ixy="0.0" ixz="0.0" -->
-	  <!-- 		   iyy="0.29" iyz="0.0" izz="0.371"/> -->
-	  <inertia ixx = "0.042" ixy = "0.0" ixz = "0.0"
-	  		   iyy = "0.142" iyz = "0.0" izz = "0.167"/>
+	  <!-- The inertia is wrong, but it's on purpose: when I fix the
+		   inertia to account for the robot's new mass value, it begins to wobble.
+		   Hence, I'll look further into it, but for now I'll leave it as is -->
+	  <inertia ixx = "0.1" ixy = "0.0" ixz = "0.0"
+	  		   iyy = "0.1" iyz = "0.0" izz = "0.1"/>
 	</inertial>
 	<!-- Front Caster -->

Commit message: Change a few colors on gazebo

File: urdf/dd_robot.xacro (robot description, xacro)
@@ -42,5 +42,5 @@
 		<sphere radius="0.05"/>
 	  </geometry>
-	  <material name="blue"/>
+	  <material name="white"/>
 	</visual>
 	<!-- Caster collision -->

File: urdf/gazebo.xacro (robot description, xacro)
@@ -6,11 +6,14 @@
   </gazebo>
   <gazebo reference="left_wheel">
-	<material>Gazebo/White</material>
+	<material>Gazebo/Orange</material>
   </gazebo>
   <gazebo reference="right_wheel">
-	<material>Gazebo/White</material>
+	<material>Gazebo/Orange</material>
   </gazebo>
   <gazebo reference="laser_scanner">
 	<material>Gazebo/Black</material>
+  </gazebo>
+  <gazebo reference="camera_link">
+	<material>Gazebo/Orange</material>
   </gazebo>
   <gazebo>

Commit message: Minor change: fixed the green color material description

File: urdf/dd_robot.xacro (robot description, xacro)
@@ -42,5 +42,5 @@
 		<sphere radius="0.05"/>
 	  </geometry>
-	  <material name="white"/>
+	  <material name="blue"/>
 	</visual>
 	<!-- Caster collision -->

File: urdf/materials.xacro (robot description, xacro)
@@ -11,5 +11,5 @@
   </material>
   <material name="green">
-	<color rgba="0.05 1.0 0.05"/>
+	<color rgba="0.05 1.0 0.05 1.0"/>
   </material>
 </robot>
